File: Control/control_module.sch (KiCad schematic (older format))
At the start: 88 parts, among them P1 CONN_02X03, P2 CONN_02X03, P3 CONN_01X04, P4 CONN_02X02, P5 CONN_02X02, P6 CONN_01X04, P7 CONN_01X02, P8 CONN_01X04, P9 CONN_01X02, Q1 Q_NMOS_GDS, Q2 Q_NMOS_GDS, Q3 IRF540N, U1 UCC3818, U2 1EDI60N12AF, U3 LM358N

Commit message: Kontrol karti semasi cizildi. Layout yerlestirme yapildi.
Parts:
- removed C1: 100u, Capacitors_SMD:CP_Elec_8x10, symbol CP1_Small
- removed C14, C29: 10n, Capacitors_SMD:C_0805_HandSoldering, symbol C_Small
- removed C15, C19: 250u, NamchoLibs:C_MKP_Vishay_70x65x57.5, symbol C
- removed C16, C28: 1u, Capacitors_SMD:C_1206_HandSoldering, symbol C_Small
- removed C17, C18, C20: C_Small, Capacitors_SMD:C_0805_HandSoldering, symbol C_Small
- removed C2: 100n, Capacitors_SMD:C_0805_HandSoldering, symbol C_Small
- removed C3: C, Capacitors_ThroughHole:C_Rect_L10.0mm_W4.0mm_P7.50mm_MKS4, symbol C
- removed D1: CrydomM50, NamchoLibs:CrydomM50x_Fixed, symbol CrydomM50
- removed D4, D6, D8: ZENERsmall, Diodes_SMD:D_SOD-123, symbol ZENERsmall
- removed D5: IDW75E60, TO_SOT_Packages_THT:TO-247_TO-3P_Vertical, symbol IDW75E60
- removed D7: C5D50065D, TO_SOT_Packages_THT:TO-247_TO-3P_Vertical, symbol C5D50065D
- removed L1: INDUCTOR_2, NamchoLibs:OD_77.80xID_39.34xHT_25.85_Horizantal, symbol INDUCTOR_2
- removed MP1, MP2, MP3, MP4, MP5, MP6: SCREW, NamchoLibs:SCREW_3mm, symbol SCREW
- removed P1, P2: CONN_02X03, NamchoLibs:Conn_6pins_30A, symbol CONN_02X03
- removed P3, P6, P8: CONN_01X04, Pin_Headers:Pin_Header_Straight_1x04_Pitch2.54mm, symbol CONN_01X04
- removed P4, P5: CONN_02X02, NamchoLibs:Conn_4pins_15A, symbol CONN_02X02
- removed P7, P9: CONN_01X02, Pin_Headers:Pin_Header_Straight_1x02_Pitch2.54mm, symbol CONN_01X02
- removed Q1, Q2: Q_NMOS_GDS, TO_SOT_Packages_THT:TO-247_TO-3P_Vertical, symbol Q_NMOS_GDS
- removed Q3: IRF540N, TO-220, symbol IRF540N
- removed R11, R12, R8, R9: 0.003, Resistors_SMD:R_2512_HandSoldering, symbol R
- removed R14, R19, R25, R26, R27, R28, R29, R30: R_Small, Resistors_SMD:R_1206_HandSoldering, symbol R_Small
- removed R15, R20, R22, R23, R24, R33, R34, R35, R36: R_Small, Resistors_SMD:R_0805_HandSoldering, symbol R_Small
- removed R16, R17: 4R7, Resistors_SMD:R_2512_HandSoldering, symbol R
- removed R21: 0, Resistors_SMD:R_0805_HandSoldering, symbol R_Small
- removed R31, R32: 10k, Resistors_SMD:R_1206_HandSoldering, symbol R_Small
- removed U2: 1EDI60N12AF, Housings_SOIC:SOIC-8_3.9x4.9mm_Pitch1.27mm, symbol 1EDI60N12AF
- removed U3: LM358N, NamchoLibs:SOIC-8-N, symbol LM358N
- added D3: D_Zener_Small_ALT, Diodes_SMD:D_SOD-123, symbol D_Zener_Small_ALT
- added J1: Conn_02x06_Counter_Clockwise, NamchoLibs:Harwin_M55_7101242R, symbol Conn_02x06_Counter_Clockwise
- renumbered C4 to C1, C13 to C10, C5 to C2, C6 to C3, C7 to C4, C8 to C5, C9 to C6, C10 to C7, C11 to C8, C12 to C9, D2 to D1, D3 to D2, R37 to R1, R13 to R10, R1 to R2, R2 to R3, R3 to R4, R4 to R5, R5 to R6, R6 to R7, R7 to R8, R10 to R9
Connections:
- net labels added: DriveOut, Isens+, Isens-, VDD, Vinput, Vout, Vovp
- net labels removed: +12V, +15V, 15V/1, 15V/3, Bridge+, Bridge-, CrtPad, GNDA, GND_DRV1, PH1, PH2, Vout+
- wire segments 283 -> 100
- no-connect marks 6 -> 0
Other:
- note removed: "12V güç kaynağı soketi"
- note removed: "2.6A(3A secilebilir) peak değeri olan gatedriver lazim."
- note removed: "Cikis gerilim ripple degeri 20V"
- note removed: "Cikis kondasatorleri Panasonic 450V 390uF 30mmx45mm secildi."
- note removed: "Co = 200x5 600V olacak."
- note removed: "Fan Kontrol"
