File: Control/control_module.kicad_pcb (KiCad board)
At the start: 2 copper layers, 25 parts, among them J1 Conn_02x06_Counter_Clockwise, U1 UCC3818

Commit message: Kontrolcu karti icin layout islemi tamamlandi.
Parts:
- moved R7 170.3 mm to (187.1, 81.5), turned to 90 degrees
- moved C4 168.7 mm to (189.1, 81.5), turned to 90 degrees
- moved C5 168.7 mm to (185.1, 81.5), turned to 90 degrees
- moved C1 165.5 mm to (184.5, 89.5), turned to 270 degrees
- moved C3 163.9 mm to (175.5, 88.8), turned to 270 degrees
- moved R4 163.3 mm to (182.2, 88.9), turned to 270 degrees
- moved R10 162.9 mm to (185.1, 75.0), turned to 270 degrees
- moved R5 162.8 mm to (177.5, 88.8), turned to 90 degrees
- moved C2 162.2 mm to (179.5, 88.8), turned to 90 degrees
- moved C7 162.1 mm to (187.1, 74.9), turned to 90 degrees
- moved C8 161.2 mm to (189.1, 74.9), turned to 90 degrees
- moved U1 159.4 mm to (177.2, 79.3), turned to 90 degrees
- moved D1 155.7 mm to (170.5, 93.0), turned to 180 degrees
- moved D2 154.8 mm to (170.5, 88.0), turned to 180 degrees
- moved D3 153.2 mm to (169.6, 72.3), turned to 180 degrees
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Routing:
- net DriveOut: track 0.00 -> 51.3 mm, vias 0 -> 2
- net Vout: track 5.21 -> 50.6 mm, vias 1 -> 2
- net Vovp: track 0.00 -> 38.3 mm, vias 0 -> 2
- net Net-(C2-Pad2): track 0.00 -> 36.2 mm, vias 0 -> 2
- net GNDD: track 0.00 -> 35.6 mm, vias 0 -> 13
- net Net-(R3-Pad1): track 0.00 -> 31.9 mm, vias 0 -> 2
- net Vref: track 0.00 -> 26.0 mm, vias 0 -> 2
- net VDD: track 0.00 -> 22.3 mm
- net Net-(D2-Pad3): track 0.00 -> 18.9 mm
- net Net-(C8-Pad2): track 0.00 -> 18.6 mm
- net Net-(R6-Pad1): track 0.00 -> 18.2 mm, vias 0 -> 2
- net Net-(C4-Pad1): track 0.00 -> 15.2 mm
- net Net-(C7-Pad2): track 0.00 -> 14.5 mm
- net Net-(R10-Pad1): track 0.00 -> 10.1 mm
- net Vinput: track 0.00 -> 8.59 mm
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- added copper zone on B.Cu, net GNDD
- added copper zone on F.Cu, net GNDD
- added copper zone on F.Cu, net Isens-
- added copper zone on F.Cu, net Net-(C1-Pad1)
- added copper zone on F.Cu, net VDD
- added copper zone on F.Cu, net Vout
Other:
- board outline added: 42 x 25 mm
- net class Bridge removed
- net class Default: clearance 0.3 -> 0.2; trace_width 0.25 -> 0.4
- net class GNDA removed
- net class Phase removed
- net class PowerTraces removed
- rule trace_clearance: 0.3 -> 0.2
- board text added: "Controller"

Commit message: Kontrol karti gerber dosyalari olusturuldu. Silk katmani duzenlendi.
Routing:
- net GNDD: vias 13 -> 9
- net (no net): vias 0 -> 4
Changed lines of the file:
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@@
   (general
     (links 48)
-    (no_connects 1)
-    (area 148.735 70.699999 211.77143 121.575)
+    (no_connects 0)
+    (area 146.235 69.225 206.05 102.000001)
     (thickness 1.6)
     (drawings 7)
@@
     (pad_to_mask_clearance 0)
     (aux_axis_origin 0 0)
-    (visible_elements 7FFCFFFF)
+    (visible_elements 7FFEFFFF)
     (pcbplotparams
       (layerselection 0x00030_80000001)
@@
     (tags "capacitor 0805")
     (attr smd)
-    (fp_text reference C8 (at 0 -1.75 90) (layer F.SilkS)
+    (fp_text reference C8 (at 2.9 0 90) (layer F.SilkS)
       (effects (font (size 1 1) (thickness 0.15)))
     )
@@
     (tags "SOIC 1.27")
     (attr smd)
-    (fp_text reference U1 (at 0 -6.25 90) (layer F.SilkS)
+    (fp_text reference U1 (at 4.65 -5.65 180) (layer F.SilkS)
       (effects (font (size 1 1) (thickness 0.15)))
     )
@@
     (tags "capacitor 1206")
     (attr smd)
-    (fp_text reference C1 (at 0 -1.75 270) (layer F.SilkS)
+    (fp_text reference C1 (at -0.578 -3.038 270) (layer F.SilkS)
       (effects (font (size 1 1) (thickness 0.15)))
     )
@@
     (tags "capacitor 0805")
     (attr smd)
-    (fp_text reference C2 (at 0 -1.75 90) (layer F.SilkS)
+    (fp_text reference C2 (at -3 0 90) (layer F.SilkS)
       (effects (font (size 1 1) (thickness 0.15)))
     )
@@
     (tags "capacitor 0805")
     (attr smd)
-    (fp_text reference C3 (at 0 -1.75 270) (layer F.SilkS)
+    (fp_text reference C3 (at 3 0 270) (layer F.SilkS)
       (effects (font (size 1 1) (thickness 0.15)))
     )
@@
     (tags "capacitor 0805")
     (attr smd)
-    (fp_text reference C4 (at 0 -1.75 90) (layer F.SilkS)
+    (fp_text reference C4 (at -3.05 0 90) (layer F.SilkS)
       (effects (font (size 1 1) (thickness 0.15)))
     )
@@
     (tags "capacitor 0805")
     (attr smd)
-    (fp_text reference C5 (at 0 -1.75 90) (layer F.SilkS)
+    (fp_text reference C5 (at -3.05 0 90) (layer F.SilkS)
       (effects (font (size 1 1) (thickness 0.15)))
     )
@@
     (tags "capacitor 1206")
     (attr smd)
-    (fp_text reference C6 (at 0 -1.75 180) (layer F.SilkS)
+    (fp_text reference C6 (at 4.05 0 180) (layer F.SilkS)
       (effects (font (size 1 1) (thickness 0.15)))
     )
@@
     (tags "capacitor 0805")
     (attr smd)
-    (fp_text reference C7 (at 0 -1.75 90) (layer F.SilkS)
+    (fp_text reference C7 (at 3 0 90) (layer F.SilkS)
       (effects (font (size 1 1) (thickness 0.15)))
     )
@@
     (tags "capacitor 1206")
     (attr smd)
-    (fp_text reference C9 (at 0 -1.75 270) (layer F.SilkS)
+    (fp_text reference C9 (at -4.05 0.05 270) (layer F.SilkS)
       (effects (font (size 1 1) (thickness 0.15)))
     )
@@
     (descr "SMT capacitor, aluminium electrolytic, 8x10")
     (attr smd)
-    (fp_text reference C10 (at 0 5.45 270) (layer F.SilkS)
+    (fp_text reference C10 (at -2.204 4.9 270) (layer F.SilkS)
       (effects (font (size 1 1) (thickness 0.15)))
     )
@@
     (tags SOT-23)
     (attr smd)
-    (fp_text reference D1 (at 0 -2.5 180) (layer F.SilkS)
+    (fp_text reference D1 (at 1.65 1.2 180) (layer F.SilkS)
       (effects (font (size 1 1) (thickness 0.15)))
     )
@@
     (tags SOT-23)
     (attr smd)
-    (fp_text reference D2 (at 0 -2.5 180) (layer F.SilkS)
+    (fp_text reference D2 (at 1.9 -1.2 180) (layer F.SilkS)
       (effects (font (size 1 1) (thickness 0.15)))
     )
@@
     (tags SOD-123)
     (attr smd)
-    (fp_text reference D3 (at 0 -2 180) (layer F.SilkS)
+    (fp_text reference D3 (at -3.3 0.55 180) (layer F.SilkS)
       (effects (font (size 1 1) (thickness 0.15)))
     )
@@
   (module NamchoLibs:Harwin_M55_7101242R placed (layer F.Cu)
     (at 153.21 87.5 270)
-    (fp_text reference J1 (at 3.5 -5.5 270) (layer F.SilkS)
+    (fp_text reference J1 (at 6.7 -5.34 270) (layer F.SilkS)
       (effects (font (size 1 1) (thickness 0.15)))
     )
@@
     (tags "resistor 0805")
     (attr smd)
-    (fp_text reference R1 (at 0 -1.7 180) (layer F.SilkS)
+    (fp_text reference R1 (at -3 0 180) (layer F.SilkS)
       (effects (font (size 1 1) (thickness 0.15)))
     )
@@
     (tags "resistor 1206")
     (attr smd)
-    (fp_text reference R3 (at 0 -1.85 180) (layer F.SilkS)
+    (fp_text reference R3 (at 0 1.65 180) (layer F.SilkS)
       (effects (font (size 1 1) (thickness 0.15)))
     )
@@
     (tags "resistor 0805")
     (attr smd)
-    (fp_text reference R4 (at 0 -1.7 270) (layer F.SilkS)
+    (fp_text reference R4 (at -0.043 -4.024 270) (layer F.SilkS)
       (effects (font (size 1 1) (thickness 0.15)))
     )
@@
     (tags "resistor 0805")
     (attr smd)
-    (fp_text reference R5 (at 0 -1.7 90) (layer F.SilkS)
+    (fp_text reference R5 (at -3.1 0 90) (layer F.SilkS)
       (effects (font (size 1 1) (thickness 0.15)))
     )
@@
     (tags "resistor 0805")
     (attr smd)
-    (fp_text reference R6 (at 0 -1.7 180) (layer F.SilkS)
+    (fp_text reference R6 (at -3 0 180) (layer F.SilkS)
       (effects (font (size 1 1) (thickness 0.15)))
     )
@@
     (tags "resistor 0805")
     (attr smd)
-    (fp_text reference R7 (at 0 -1.7 90) (layer F.SilkS)
+    (fp_text reference R7 (at -3.1 0 90) (layer F.SilkS)
       (effects (font (size 1 1) (thickness 0.15)))
     )
@@
     (tags "resistor 0805")
     (attr smd)
-    (fp_text reference R8 (at 0 -1.7) (layer F.SilkS)
+    (fp_text reference R8 (at 3.05 0) (layer F.SilkS)
       (effects (font (size 1 1) (thickness 0.15)))
     )
@@
     (tags "resistor 0805")
     (attr smd)
-    (fp_text reference R9 (at 0 -1.7) (layer F.SilkS)
+    (fp_text reference R9 (at -3.15 0) (layer F.SilkS)
       (effects (font (size 1 1) (thickness 0.15)))
     )
@@
     (tags "resistor 0805")
     (attr smd)
-    (fp_text reference R10 (at 0 -1.7 270) (layer F.SilkS)
+    (fp_text reference R10 (at 0 1.55 270) (layer F.SilkS)
       (effects (font (size 1 1) (thickness 0.15)))
     )
@@
     )
   )
-  (gr_text Controller (at 182.2 94.2 360) (layer F.Cu)
+  (gr_text Controller (at 182.2 94.2) (layer F.Cu)
     (effects (font (size 1.5 1.5) (thickness 0.3)))
   )
@@
   (gr_line (start 148.5 70.5) (end 148.5 95.5) (angle 90) (layer Edge.Cuts) (width 0.1))
   (gr_line (start 190.5 70.5) (end 148.5 70.5) (angle 90) (layer Edge.Cuts) (width 0.1))
+  (via (at 186.2 77.4) (size 0.6) (drill 0.4) (layers F.Cu B.Cu) (net 0))
+  (via (at 187.8 77.4) (size 0.6) (drill 0.4) (layers F.Cu B.Cu) (net 0))
+  (via (at 169 80.25) (size 0.6) (drill 0.4) (layers F.Cu B.Cu) (net 0))
+  (via (at 169.75 80.25) (size 0.6) (drill 0.4) (layers F.Cu B.Cu) (net 0))
   (segment (start 182.226 86.326) (end 181.645 85.745) (width 0.4) (layer F.Cu) (net 1))
   (segment (start 181.645 85.745) (end 181.645 83.95) (width 0.4) (layer F.Cu) (net 1))
@@
   (segment (start 171.655 81.7) (end 172.355 82.4) (width 0.8) (layer F.Cu) (net 2))
   (segment (start 170.2 81.7) (end 171.655 81.7) (width 0.8) (layer F.Cu) (net 2))
-  (via (at 186.2 77.4) (size 0.6) (drill 0.4) (layers F.Cu B.Cu) (net 2))
-  (via (at 187.8 77.4) (size 0.6) (drill 0.4) (layers F.Cu B.Cu) (net 2))
   (segment (start 187.1 77.3) (end 187 77.4) (width 0.6) (layer F.Cu) (net 2))
   (via (at 187 77.4) (size 0.6) (drill 0.4) (layers F.Cu B.Cu) (net 2))
@@
   (segment (start 182.226 91.426) (end 182.6 91.8) (width 1) (layer F.Cu) (net 2))
   (via (at 182.6 91.8) (size 0.6) (drill 0.4) (layers F.Cu B.Cu) (net 2))
-  (via (at 169 80.25) (size 0.6) (drill 0.4) (layers F.Cu B.Cu) (net 2))
-  (via (at 169.75 80.25) (size 0.6) (drill 0.4) (layers F.Cu B.Cu) (net 2))
   (segment (start 170.2 81.7) (end 170.2 80.55) (width 0.4) (layer F.Cu) (net 2))
   (segment (start 170.2 80.55) (end 170.5 80.25) (width 0.4) (layer F.Cu) (net 2))
